Commit message: Just added pure pursuit with move_base path planning. Want to back up all the system level racecar config files

File: src/simulator/racecar-simulator/racecar_description/urdf/macros.xacro (robot description, xacro)
@@ -4,5 +4,5 @@
 <xacro:macro name="chassis_inertial_params">
   <origin xyz="0.1477 0 0" rpy="0 0 0" />
-  <mass value="4.0" />
+  <mass value="10.0" />
   <inertia ixx="0.010609" ixy="0"          ixz="0"
                           iyy="0.050409"   iyz="0"

File: src/simulator/racecar-simulator/racecar_description/urdf/racecar.xacro (robot description, xacro)
@@ -43,5 +43,5 @@
     <child link="left_rear_wheel" />
     <axis xyz="0 0 -1" />
-    <limit effort="10" velocity="100" />
+    <limit effort="10" velocity="1000" />
   </joint>
   <xacro:wheel_transmission name="left_rear_wheel" />
@@ -64,5 +64,5 @@
     <child link="right_rear_wheel" />
     <axis xyz="0 0 -1" />
-    <limit effort="10" velocity="100" />
+    <limit effort="10" velocity="1000" />
   </joint>
   <xacro:wheel_transmission name="right_rear_wheel" />
@@ -82,5 +82,5 @@
     <child link="left_steering_hinge" />
     <axis xyz="-1 0 0" />
-    <limit lower="-1.0" upper="1.0" effort="10" velocity="100" />
+    <limit lower="-1.0" upper="1.0" effort="10" velocity="1000" />
   </joint>
   <xacro:steering_hinge_transmission name="left_steering_hinge" />
@@ -100,5 +100,5 @@
     <child link="right_steering_hinge" />
     <axis xyz="-1 0 0" />
-    <limit lower="-1.0" upper="1.0" effort="10" velocity="100" />
+    <limit lower="-1.0" upper="1.0" effort="10" velocity="1000" />
   </joint>
   <xacro:steering_hinge_transmission name="right_steering_hinge" />
@@ -121,5 +121,5 @@
     <child link="left_front_wheel" />
     <axis xyz="0 0 -1" />
-    <limit effort="10" velocity="100" />
+    <limit effort="10" velocity="1000" />
   </joint>
   <xacro:wheel_transmission name="left_front_wheel" />
@@ -142,5 +142,5 @@
     <child link="right_front_wheel" />
     <axis xyz="0 0 -1" />
-    <limit effort="10" velocity="100"/>
+    <limit effort="10" velocity="1000"/>
   </joint>
   <xacro:wheel_transmission name="right_front_wheel" />
